Commit message: RL control

File: src/rr100_description/urdf/chassis_rr100.urdf.xacro (robot description, xacro)
@@ -18,5 +18,5 @@
     <link name="base_link">
       <visual>
-        <origin xyz="0.03 0 -0.1" rpy="0 ${-M_PI/2} 0" />
+        <origin xyz="0 0 -0.1" rpy="0 ${-M_PI/2} 0" />
         <geometry>
           <mesh filename="package://rr100_description/meshes/rr100.dae" scale="0.001 0.001 0.001" />
@@ -25,5 +25,5 @@
       </visual>
       <collision>
-        <origin xyz="0.03 0 -0.1" rpy="0 ${-M_PI/2} 0" />
+        <origin xyz="0 0 -0.1" rpy="0 ${-M_PI/2} 0" />
         <geometry>
           <mesh filename="package://rr100_description/meshes/rr100.dae" scale="0.001 0.001 0.001" />

File: src/rr100_description/urdf/rr100.urdf.xacro (robot description, xacro)
@@ -17,6 +17,6 @@
   <xacro:property name="wheel_x_offset" value="0.0" />
   <xacro:property name="wheel_y_offset" value="0.0" />
-  <xacro:property name="wheelbase" value="0.600" />
-  <xacro:property name="track" value="0.500" />
+  <xacro:property name="wheelbase" value="0.500" />
+  <xacro:property name="track" value="0.600" />
   <xacro:chassis/>
   <!-- Wheel macros -->
@@ -55,5 +55,5 @@
     <xacro:include filename="$(find robosense_description)/urdf/RS-16.urdf.xacro"/>
     <xacro:RS-16 parent="base_link" name="rslidar" topic="/rslidar_points" hz="20" samples="2625" gpu="${gpu}">
-        <origin xyz="0.032 0 0.40" rpy="0.0 0.0 0.0" />
+        <origin xyz="0 0 0.416" rpy="0.0 0.0 0.0" />
     </xacro:RS-16>
   </xacro:if>
